File: hw/shoulder.sch (KiCad schematic (older format))
At the start: 27 parts, among them J1 IDC_02X07, U1 OSRB38C9BA, U2 OSRB38C9BA, U3 OSRB38C9BA, U4 OSRB38C9BA, U5 OSRB38C9BA

Commit message: updated schematic
Parts:
- D1, D2: footprint LED_SMD:LED_WS2812-PLCC6 -> KLIB_Opto:LED_RGB_5050-6
- U1, U2, U3, U4: footprint KLIB_Opto:OSRB8C9BA -> KLIB_Opto:OSRB8C9BA_Vertical
- U5: footprint KLIB_Opto:OSRB8C9BA-90 -> KLIB_Opto:OSRB8C9BA_Vertical
Connections:
- net REP+ is gone; now on net SP+: J1.13
- net REP- is gone; now on net SP-: J1.12
- net SP+: now reaches LS1.1 (+)
- net SP-: now reaches LS1.2 (-)
Other:
- moved on the sheet: J1, LS1

Commit message: updated schematic
Parts:
- R1, R10, R11, R2, R3, R4, R5, R6, R7, R8, R9: footprint Resistor_SMD:R_0805_2012Metric_Pad1.15x1.50mm_HandSolder -> Resistor_SMD:R_0805_2012Metric
- U5: footprint KLIB_Opto:OSRB8C9BA_Vertical -> KLIB_Opto:OSRB8C9BA_Horizontal
Changed lines of the file:
@@
 F 0 "R6" H 4220 3446 50  0000 L CNN
 F 1 "120R" H 4220 3355 50  0000 L CNN
-F 2 "Resistor_SMD:R_0805_2012Metric_Pad1.15x1.50mm_HandSolder" V 4080 3400 50  0001 C CNN
+F 2 "Resistor_SMD:R_0805_2012Metric" V 4080 3400 50  0001 C CNN
 F 3 "" H 4150 3400 50  0001 C CNN
 	1    4150 3400
@@
 F 0 "R7" H 4620 3446 50  0000 L CNN
 F 1 "120R" H 4620 3355 50  0000 L CNN
-F 2 "Resistor_SMD:R_0805_2012Metric_Pad1.15x1.50mm_HandSolder" V 4480 3400 50  0001 C CNN
+F 2 "Resistor_SMD:R_0805_2012Metric" V 4480 3400 50  0001 C CNN
 F 3 "" H 4550 3400 50  0001 C CNN
 	1    4550 3400
@@
 F 0 "R8" H 5020 3446 50  0000 L CNN
 F 1 "180R" H 5020 3355 50  0000 L CNN
-F 2 "Resistor_SMD:R_0805_2012Metric_Pad1.15x1.50mm_HandSolder" V 4880 3400 50  0001 C CNN
+F 2 "Resistor_SMD:R_0805_2012Metric" V 4880 3400 50  0001 C CNN
 F 3 "" H 4950 3400 50  0001 C CNN
 	1    4950 3400
@@
 F 0 "R1" H 1520 1146 50  0000 L CNN
 F 1 "100R" H 1520 1055 50  0000 L CNN
-F 2 "Resistor_SMD:R_0805_2012Metric_Pad1.15x1.50mm_HandSolder" V 1380 1100 50  0001 C CNN
+F 2 "Resistor_SMD:R_0805_2012Metric" V 1380 1100 50  0001 C CNN
 F 3 "" H 1450 1100 50  0001 C CNN
 	1    1450 1100
@@
 F 0 "R2" H 1520 2496 50  0000 L CNN
 F 1 "100R" H 1520 2405 50  0000 L CNN
-F 2 "Resistor_SMD:R_0805_2012Metric_Pad1.15x1.50mm_HandSolder" V 1380 2450 50  0001 C CNN
+F 2 "Resistor_SMD:R_0805_2012Metric" V 1380 2450 50  0001 C CNN
 F 3 "" H 1450 2450 50  0001 C CNN
 	1    1450 2450
@@
 F 0 "R3" H 1520 3846 50  0000 L CNN
 F 1 "100R" H 1520 3755 50  0000 L CNN
-F 2 "Resistor_SMD:R_0805_2012Metric_Pad1.15x1.50mm_HandSolder" V 1380 3800 50  0001 C CNN
+F 2 "Resistor_SMD:R_0805_2012Metric" V 1380 3800 50  0001 C CNN
 F 3 "" H 1450 3800 50  0001 C CNN
 	1    1450 3800
@@
 F 0 "R4" H 3320 1146 50  0000 L CNN
 F 1 "100R" H 3320 1055 50  0000 L CNN
-F 2 "Resistor_SMD:R_0805_2012Metric_Pad1.15x1.50mm_HandSolder" V 3180 1100 50  0001 C CNN
+F 2 "Resistor_SMD:R_0805_2012Metric" V 3180 1100 50  0001 C CNN
 F 3 "" H 3250 1100 50  0001 C CNN
 	1    3250 1100
@@
 F 0 "R5" H 3320 2496 50  0000 L CNN
 F 1 "100R" H 3320 2405 50  0000 L CNN
-F 2 "Resistor_SMD:R_0805_2012Metric_Pad1.15x1.50mm_HandSolder" V 3180 2450 50  0001 C CNN
+F 2 "Resistor_SMD:R_0805_2012Metric" V 3180 2450 50  0001 C CNN
 F 3 "" H 3250 2450 50  0001 C CNN
 	1    3250 2450
@@
 F 0 "R9" H 6120 3446 50  0000 L CNN
 F 1 "120R" H 6120 3355 50  0000 L CNN
-F 2 "Resistor_SMD:R_0805_2012Metric_Pad1.15x1.50mm_HandSolder" V 5980 3400 50  0001 C CNN
+F 2 "Resistor_SMD:R_0805_2012Metric" V 5980 3400 50  0001 C CNN
 F 3 "" H 6050 3400 50  0001 C CNN
 	1    6050 3400
@@
 F 0 "R10" H 6520 3446 50  0000 L CNN
 F 1 "120R" H 6520 3355 50  0000 L CNN
-F 2 "Resistor_SMD:R_0805_2012Metric_Pad1.15x1.50mm_HandSolder" V 6380 3400 50  0001 C CNN
+F 2 "Resistor_SMD:R_0805_2012Metric" V 6380 3400 50  0001 C CNN
 F 3 "" H 6450 3400 50  0001 C CNN
 	1    6450 3400
@@
 F 0 "R11" H 6920 3446 50  0000 L CNN
 F 1 "180R" H 6920 3355 50  0000 L CNN
-F 2 "Resistor_SMD:R_0805_2012Metric_Pad1.15x1.50mm_HandSolder" V 6780 3400 50  0001 C CNN
+F 2 "Resistor_SMD:R_0805_2012Metric" V 6780 3400 50  0001 C CNN
 F 3 "" H 6850 3400 50  0001 C CNN
 	1    6850 3400
@@
 F 0 "U5" H 2726 3117 50  0000 C CNN
 F 1 "OSRB38C9BA" H 2726 3026 50  0000 C CNN
-F 2 "KLIB_Opto:OSRB8C9BA_Vertical" H 2750 2400 50  0001 C CNN
+F 2 "KLIB_Opto:OSRB8C9BA_Horizontal" H 2750 2400 50  0001 C CNN
 F 3 "http://www.tme.eu/cz/Document/777fdf21e0fba3fd5c036ef95756460c/OSRB38C9BA.pdf" H 2800 2400 50  0001 C CNN
 	1    2750 2750
